File: HackPad/HackPad.kicad_pcb (KiCad board)
At the start: 2 copper layers, 100 x 100 mm, 19 parts, among them SW1 SW_Push, SW10 SW_Push, SW11 SW_Push, SW12 SW_Push, SW13 SW_Push, SW14 SW_Push, SW15 SW_Push, SW16 SW_Push, SW2 SW_Push, SW3 SW_Push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

Commit message: gerber
Parts:
- removed RV1, RV2: R_Potentiometer, Potentiometer_THT:Potentiometer_Alps_RK09L_Single_Vertical
- removed SW10, SW11, SW12, SW13, SW14, SW15, SW16, SW9: SW_Push, Button_Switch_Keyboard:SW_Cherry_MX_1.00u_PCB
- added H1: MountingHole, MountingHole:MountingHole_3.2mm_M3, F.Cu at (54.2, 41.0)
- added H2: MountingHole, MountingHole:MountingHole_3.2mm_M3, F.Cu at (140.2, 40.8)
- added H3: MountingHole, MountingHole:MountingHole_3.2mm_M3, F.Cu at (69.5, 83.0)
- added H4: MountingHole, MountingHole:MountingHole_3.2mm_M3, F.Cu at (120.0, 72.5)
- SW7: value SW_Push -> RotaryEncoder_Switch; footprint Button_Switch_Keyboard:SW_Cherry_MX_1.00u_PCB -> Rotary_Encoder:RotaryEncoder_Alps_EC11E-Switch_Vertical_H20mm
- SW8: value SW_Push -> RotaryEncoder; footprint Button_Switch_Keyboard:SW_Cherry_MX_1.00u_PCB -> Rotary_Encoder:RotaryEncoder_Alps_EC11E-Switch_Vertical_H20mm
- U1: moved to F.Cu
- moved SW7 72.2 mm to (132.0, 51.2)
- moved SW8 71.7 mm to (132.0, 71.0)
- moved SW3 56.6 mm to (81.4, 48.9)
- moved SW4 56.6 mm to (81.4, 67.9)
- moved SW5 46.8 mm to (100.5, 48.9), turned to 0 degrees
- moved SW6 24.9 mm to (100.5, 67.9)
- moved U1 18.7 mm to (118.9, 46.4), turned to 0 degrees
- moved SW2 14.8 mm to (62.4, 67.9)
- moved SW1 14.8 mm to (62.4, 48.9)
Connections:
- SW1 pad 2: Net-(U1-PA6_A10_D10_MOSI) -> GND
- SW2 pad 2: Net-(U1-PA6_A10_D10_MOSI) -> GND
- SW3 pad 2: Net-(U1-PA6_A10_D10_MOSI) -> GND
- SW4 pad 2: Net-(U1-PA6_A10_D10_MOSI) -> GND
- SW5 pad 1: Net-(U1-PA6_A10_D10_MOSI) -> Net-(U1-PA7_A8_D8_SCK)
- SW5 pad 2: Net-(U1-PA5_A9_D9_MISO) -> GND
- SW6 pad 1: Net-(U1-PA6_A10_D10_MOSI) -> Net-(U1-PB09_A7_D7_RX)
- SW6 pad 2: Net-(U1-PA5_A9_D9_MISO) -> GND
- U1 pad 13: /GND -> GND
- U1 pad 7: unconnected-(U1-PB08_A6_D6_TX-Pad7) -> Net-(U1-PB08_A6_D6_TX)
Routing:
- net GND: track 0.00 -> 199.3 mm
- net Net-(U1-PA6_A10_D10_MOSI): track 218.6 -> 32.8 mm
- net Net-(U1-PA5_A9_D9_MISO): track 193.6 -> 30.8 mm
- net Net-(U1-PA7_A8_D8_SCK): track 159.5 -> 34.8 mm, vias 0 -> 1
- net /PWR: track 119.4 -> 0.00 mm, vias 2 -> 0
- net Net-(U1-PA10_A2_D2): track 136.9 -> 31.9 mm, vias 1 -> 0
- net /GND: track 100.4 -> 0.00 mm
- net Net-(U1-PA11_A3_D3): track 147.5 -> 48.7 mm
- net Net-(U1-PA9_A5_D5_SCL): track 84.1 -> 22.7 mm
- net Net-(U1-PA4_A1_D1): track 130.7 -> 69.4 mm
- net Net-(U1-PB09_A7_D7_RX): track 89.5 -> 38.5 mm
- net Net-(U1-PA02_A0_D0): track 101.2 -> 53.1 mm, vias 1 -> 0
- net Net-(U1-PA8_A4_D4_SDA): track 67.6 -> 21.7 mm
- net Net-(U1-PB08_A6_D6_TX): track 0.00 -> 37.3 mm
Other:
- board size 100 x 100 mm -> 100 x 51.7 mm
- board text added: "Goblin"
- board text added: "HACKPAD"

Commit message: final build with updated code and schematics
Parts:
- removed SW5, SW6: SW_Push, Button_Switch_Keyboard:SW_Cherry_MX_1.00u_PCB
- removed SW8: RotaryEncoder, Rotary_Encoder:RotaryEncoder_Alps_EC11E-Switch_Vertical_H20mm
- moved U1 6.25 mm to (112.6, 46.4)
Connections:
- net GND renamed /GND
- U1 pad 10: Net-(U1-PA5_A9_D9_MISO) -> unconnected-(U1-PA5_A9_D9_MISO-Pad10)
- U1 pad 11: Net-(U1-PA6_A10_D10_MOSI) -> unconnected-(U1-PA6_A10_D10_MOSI-Pad11)
- U1 pad 8: Net-(U1-PB09_A7_D7_RX) -> unconnected-(U1-PB09_A7_D7_RX-Pad8)
- U1 pad 9: Net-(U1-PA7_A8_D8_SCK) -> unconnected-(U1-PA7_A8_D8_SCK-Pad9)
Routing:
- net /GND: track 199.3 -> 150.9 mm
- net Net-(U1-PB09_A7_D7_RX): track 38.5 -> 0.00 mm, vias 1 -> 0
- net Net-(U1-PA7_A8_D8_SCK): track 34.8 -> 0.00 mm, vias 1 -> 0
- net Net-(U1-PA6_A10_D10_MOSI): track 32.8 -> 0.00 mm
- net Net-(U1-PA5_A9_D9_MISO): track 30.8 -> 0.00 mm, vias 1 -> 0
- net Net-(U1-PA8_A4_D4_SDA): track 21.7 -> 28.9 mm
- net Net-(U1-PB08_A6_D6_TX): track 37.3 -> 43.5 mm
- net Net-(U1-PA9_A5_D5_SCL): track 22.7 -> 29.0 mm
- net Net-(U1-PA10_A2_D2): track 31.9 -> 25.7 mm
- net Net-(U1-PA02_A0_D0): track 53.1 -> 46.9 mm
- net Net-(U1-PA4_A1_D1): track 69.4 -> 63.4 mm
- net Net-(U1-PA11_A3_D3): track 48.7 -> 44.6 mm
