File: HackPad/HackPad.kicad_sch (KiCad schematic)
At the start: 19 parts, among them SW1 SW_Push, SW10 SW_Push, SW11 SW_Push, SW12 SW_Push, SW13 SW_Push, SW14 SW_Push, SW15 SW_Push, SW16 SW_Push, SW2 SW_Push, SW3 SW_Push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

Commit message: gerber
Parts:
- removed RV1, RV2: R_Potentiometer, Potentiometer_THT:Potentiometer_Alps_RK09L_Single_Vertical, symbol Device:R_Potentiometer
- removed SW10, SW11, SW12, SW13, SW14, SW15, SW16, SW7, SW8, SW9: SW_Push, Button_Switch_Keyboard:SW_Cherry_MX_1.00u_PCB, symbol Switch:SW_Push
- added H1, H2, H3, H4: MountingHole, MountingHole:MountingHole_3.2mm_M3, symbol Mechanical:MountingHole
- added SW7: RotaryEncoder_Switch, Rotary_Encoder:RotaryEncoder_Alps_EC11E-Switch_Vertical_H20mm, symbol Device:RotaryEncoder_Switch
- added SW8: RotaryEncoder, Rotary_Encoder:RotaryEncoder_Alps_EC11E-Switch_Vertical_H20mm, symbol Device:RotaryEncoder
Connections:
- net GND: now also SW1.2, SW2.2, SW3.2, SW4.2, SW5.2, SW6.2, SW7.C, SW7.S2, SW8.C
- net at U1.9 (PA7_A8_D8_SCK): now also SW5.1
- net at U1.8 (PB09_A7_D7_RX): now also SW6.1
- net at U1.5 (PA8_A4_D4_SDA): now also SW7.A
- net at U1.6 (PA9_A5_D5_SCL): now also SW7.B
- net at U1.7 (PB08_A6_D6_TX): now also SW7.S1
- new net: SW8.A, U1.10 (PA5_A9_D9_MISO)
- new net: SW8.B, U1.11 (PA6_A10_D10_MOSI)
- no-connect marks 0 -> 1

Commit message: final build with updated code and schematics
Parts:
- removed SW5, SW6: SW_Push, Button_Switch_Keyboard:SW_Cherry_MX_1.00u_PCB, symbol Switch:SW_Push
- removed SW8: RotaryEncoder, Rotary_Encoder:RotaryEncoder_Alps_EC11E-Switch_Vertical_H20mm, symbol Device:RotaryEncoder
Connections:
- no-connect marks 1 -> 5
Other:
- moved on the sheet: SW1, SW2, SW3, SW4
